File: ginger-micro-board/notes.kicad_sch (KiCad schematic)
At the start: 0 parts

Commit message: changed sheet title
Other:
- title: OpenForge Cover Page -> ginger-micro-board Cover Page
Changed lines of the file:
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@@
 	(paper "B")
 	(title_block
-		(title "OpenForge Cover Page")
+		(title "ginger-micro-board Cover Page")
 	)
 	(text_box "3"
